File: Client-Files/10 - Manley VS-MU - 21-June-2025/Manley-VS-MU.kicad_pcb (KiCad board)
At the start: 2 copper layers, 455 x 88.9 mm, 104 parts, among them SW1 SW_Rotary_1x5_MP, SW2 SW_Rotary_1x5_MP

Commit message: Design_files folder added
Parts:
- moved ESP32-S3-1 50.7 mm to (185.6, 153.4), turned to -90 degrees
- moved C20 27.3 mm to (199.0, 121.5)
- moved C21 27.3 mm to (210.0, 116.5)
- moved C22 27.3 mm to (210.0, 118.0)
- moved C7 27.3 mm to (211.0, 128.5)
- moved C8 27.3 mm to (222.0, 123.5)
- moved C9 27.3 mm to (222.0, 125.0)
- moved OpAmp1 27.3 mm to (217.5, 128.5)
- moved OpAmp2 27.3 mm to (205.5, 121.5)
- moved R18 27.3 mm to (210.3, 130.0)
- moved R30 27.3 mm to (198.3, 123.0)
- moved toggle_sw2 6.80 mm to (226.2, 142.7)
Routing:
- net 3.3V: track 1124.5 -> 1171.6 mm
- net I8: track 55.3 -> 61.9 mm
- net unconnected-(ESP32-S3-1-GPIO11/ADC2_CH0-Pad17): track 1.13 -> 0.00 mm, vias 2 -> 0
- net GND: track 57.5 -> 58.6 mm, vias 137 -> 140
- net Net-(OpAmp1A-VINA+): vias 1 -> 0
- added copper zone on F.Cu, net GND

Commit message: #1 Placement in progress
Parts:
- moved ESP32-S3-1 50.7 mm to (213.8, 111.3), turned to 180 degrees
- moved C20 27.3 mm to (196.0, 148.6)
- moved C21 27.3 mm to (207.0, 143.6)
- moved C22 27.3 mm to (207.0, 145.1)
- moved C7 27.3 mm to (208.0, 155.6)
- moved C8 27.3 mm to (219.0, 150.6)
- moved C9 27.3 mm to (219.0, 152.1)
- moved OpAmp1 27.3 mm to (214.5, 155.6)
- moved OpAmp2 27.3 mm to (202.5, 148.6)
- moved R18 27.3 mm to (207.3, 157.1)
- moved R30 27.3 mm to (195.3, 150.1)
- moved toggle_sw2 6.80 mm to (233.0, 142.7)
Routing:
- net 3.3V: track 1171.6 -> 1124.5 mm
- net I8: track 61.9 -> 55.3 mm
- net unconnected-(ESP32-S3-1-GPIO11/ADC2_CH0-Pad17): track 0.00 -> 1.13 mm, vias 0 -> 2
- net GND: track 58.6 -> 57.5 mm, vias 140 -> 137
- net Net-(OpAmp1A-VINA+): vias 0 -> 1
- removed copper zone on F.Cu, net GND
