File: Design_Files/10 - Manley VS-MU - 21-June-2025/Manley-VS-MU.kicad_pcb (KiCad board)
At the start: 2 copper layers, 455 x 88.9 mm, 104 parts, among them SW1 SW_Rotary_1x5_MP, SW2 SW_Rotary_1x5_MP

Commit message: #1 Routing in progress
Parts:
- moved R18 32.6 mm to (178.6, 141.6)
- moved OpAmp1 32.5 mm to (185.5, 141.0)
- moved C7 31.3 mm to (180.2, 141.2)
- moved C9 31.1 mm to (190.2, 140.2)
- moved C8 31.0 mm to (190.2, 139.0)
- moved OpAmp2 25.2 mm to (185.5, 130.0)
- moved R30 25.2 mm to (179.3, 130.6)
- moved C20 23.8 mm to (181.0, 130.1)
- moved C21 22.8 mm to (190.2, 128.2)
- moved C22 22.8 mm to (190.2, 129.7)
- moved R1 1.33 mm to (174.3, 135.0)
- moved ESP32-S3-1 0.12 mm to (212.5, 118.1)
Routing:
- net EXT_12V: track 465.3 -> 146.5 mm
- net Net-(NPN_Transistor1-C): track 338.8 -> 31.0 mm
- net VU_DRIVE: track 341.7 -> 37.3 mm, vias 2 -> 0
- net led_VU: track 406.0 -> 134.6 mm
- net REG_5V: track 139.8 -> 46.9 mm, vias 2 -> 0
- net 3.3V: track 1124.5 -> 1052.5 mm, vias 16 -> 15
- net VU_DRIVE_2: track 63.5 -> 4.68 mm, vias 2 -> 1
- net rotary_sw_2: track 230.5 -> 183.9 mm
- net VU_uC_1: track 35.1 -> 0.84 mm, vias 0 -> 1
- net VU_uC_2: track 28.9 -> 0.76 mm, vias 0 -> 1
- net Net-(ESP32-S3-1-GPIO3/ADC1_CH2): track 27.2 -> 0.00 mm, vias 1 -> 0
- net GND: track 57.5 -> 52.0 mm, vias 137 -> 131
- net Net-(OpAmp2A-VINA+): track 5.23 -> 2.94 mm
- net AUDIO_IN_1: track 5.17 -> 3.84 mm
- net (no net): track 1.13 -> 0.00 mm, vias 2 -> 0
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- removed copper zone on B.Cu, net GND
Other:
- board size 455 x 88.9 mm -> 455 x 89.1 mm

Commit message: #1 Completed
Routing:
- net Net-(NPN_Transistor1-C): track 31.0 -> 472.2 mm, vias 0 -> 3
- net EXT_12V: track 146.5 -> 584.1 mm, vias 0 -> 4
- net VU_DRIVE: track 37.3 -> 434.2 mm, vias 0 -> 2
- net led_VU: track 134.6 -> 286.1 mm
- net REG_5V: track 46.9 -> 159.6 mm, vias 0 -> 7
- net VU_uC_1: track 0.84 -> 104.1 mm, vias 1 -> 3
- net 3.3V: track 1052.5 -> 1142.2 mm, vias 15 -> 13
- net Net-(ESP32-S3-1-GPIO4/ADC1_CH3): track 23.5 -> 108.6 mm, vias 1 -> 0
- net Net-(ESP32-S3-1-GPIO3/ADC1_CH2): track 0.00 -> 84.4 mm
- net VU_uC_2: track 0.76 -> 80.0 mm, vias 1 -> 3
- net VU_DRIVE_2: track 4.68 -> 71.8 mm, vias 1 -> 2
- net RST: track 317.9 -> 364.2 mm, vias 1 -> 3
- net MISO: track 314.0 -> 348.6 mm
- net MOSI: track 300.1 -> 324.8 mm
- net S2: track 70.8 -> 87.6 mm
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- added copper zone on B.Cu, net GND
- added copper zone on F.Cu, net GND
