File: Design_Files/24 - SSL EQ Rack - 6-June-2025/SSL-EQ-Rack.kicad_pcb (KiCad board)
At the start: 4 copper layers, 455.1 x 44.4 mm, 111 parts

Commit message: #4 Completed
Parts:
- moved pot13 1.00 mm to (268.7, 118.6)
- moved C2 0.93 mm to (461.9, 98.9)
- moved R22 0.58 mm to (485.5, 104.8)
- moved C3 0.09 mm to (461.1, 108.4)
- moved ESP32-S3-1 0.06 mm to (484.8, 105.8)
Routing:
- net INT: track 400.7 -> 461.9 mm, vias 0 -> 2
- net sig_1: track 280.3 -> 340.7 mm, vias 1 -> 2
- net SER: track 131.5 -> 191.8 mm
- net CS: track 403.5 -> 460.3 mm, vias 0 -> 2
- net SCLK: track 422.7 -> 466.8 mm, vias 3 -> 5
- net RCLK_latch: track 158.8 -> 198.7 mm
- net REG_5V: track 37.0 -> 68.3 mm, vias 1 -> 3
- net RST: track 421.4 -> 447.3 mm, vias 0 -> 1
- net 3.3V: track 921.5 -> 945.5 mm
- net MOSI: track 406.3 -> 429.6 mm
- net MISO: track 419.7 -> 441.1 mm
- net EXT_12V: track 293.9 -> 313.6 mm, vias 0 -> 3
- net sig_3: track 11.0 -> 28.6 mm, vias 1 -> 2
- net S0: track 282.7 -> 292.3 mm
- net S3: track 299.6 -> 290.0 mm, vias 3 -> 4
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Other:
- outline, holes or cut-outs redrawn
